Commit message: one laser

File: ceres_description/urdf/ceres.urdf.xacro (robot description, xacro)
@@ -137,125 +137,10 @@
     xyz="${axis_back} ${axis_right} ${axis_height}" />
   <xacro:sick_tim551
-    name="front_scanner"
-    ros_topic="/front_scan"/>
-  <xacro:sick_tim551
-    name="rear_scanner"
-    ros_topic="/rear_scan"/>
-  <xacro:box_for_joint
-    name="pico_flexx_holder1"
-    r_x="0"
-    r_y="0"
-    r_z="0"
-    o_x="0"
-    o_y="0"
-    o_z="0"
-    color="silver"
-    r="0.5"
-    g="0.5"
-    b="0.5"
-    length="0.015"
-    width="0.02"
-    height="0.02" />
-  <xacro:box_for_joint
-    name="pico_flexx_holder2"
-    r_x="0"
-    r_y="0"
-    r_z="0"
-    o_x="0"
-    o_y="0"
-    o_z="0"
-    color="silver"
-    r="0.5"
-    g="0.5"
-    b="0.5"
-    length="0.015"
-    width="0.02"
-    height="0.02" />
-  <xacro:box_for_joint
-    name="pico_flexx_model"
-    r_x="0"
-    r_y="0"
-    r_z="0"
-    o_x="0"
-    o_y="0"
-    o_z="0"
-    color="black"
-    r="0"
-    g="0"
-    b="0"
-    length="0.01"
-    width="0.067"
-    height="0.02"/>
- <!--
-  <xacro:box_for_joint
-    name="pico_flexx_bottom_plate"
-    r_x="0"
-    r_y="0"
-    r_z="0"
-    color="silver"
-    r="0.5"
-    g="0.5"
-    b="0.5"
-    length="0.01"
-    width="0.065"
-    height="0.002"/>
-  /-->
-  <link name="pico_flexx_optical_frame" type="fixed">
-    <visual>
-        <origin xyz="0 0 0" rpy="0 0 0"/>
-        <geometry>
-          <cylinder length="0.004" radius="0.0035"/>
-        </geometry>
-        <material name="white">
-          <color rgba="255 255 255 1"/>
-        </material>
-    </visual>
-  </link>
-  <link name="pico_flexx_axis" type="fixed">
-    <visual>
-        <origin xyz="0 0 0" rpy="0 ${M_PI/2} ${M_PI/2}"/>
-        <geometry>
-          <cylinder length="0.02" radius="0.01"/>
-        </geometry>
-        <material name="silver">
-          <color rgba="0.6 0.6 0.5 1"/>
-        </material>
-    </visual>
-  </link>
-  <joint name="pico_flexx_holder_to_base_joint" type="fixed">
-   <parent link="base_link" />
-   <child link="pico_flexx_holder1_link"/>
-   <origin xyz="${body_length/2} 0 ${body_height/2 - 0.01}"/>
-  </joint>
-  <joint name="pico_flexx_angle" type="continuous">
-    <parent link="pico_flexx_holder1_link"/>
-    <child link="pico_flexx_axis"/>
-    <origin xyz="0.01 0 0"/>
-    <axis xyz="0 1 0"/>
-  </joint>
-  <joint name="pico_flexx" type="fixed">
-    <parent link="pico_flexx_holder2_link" />
-    <child link="pico_flexx_model_link" />
-    <origin xyz="0.005 0 0" />
-  </joint>
-  <joint name="pico_flexx_joint" type="fixed">
-    <parent link="pico_flexx_axis"/>
-    <child link="pico_flexx_holder2_link"/>
-    <origin xyz="0.01 0 0"/>
-  </joint>
-  <joint name="front_scanner_to_base_joint" type="fixed">
+    name="scanner"
+    ros_topic="/scan"/>
+  <joint name="scanner_to_base_joint" type="fixed">
     <parent link="base_link" />
-    <child link="front_scanner_mount_link" />
+    <child link="scanner_mount_link" />
     <origin xyz="${body_length/2 - 0.035} 0 ${body_height/2 - 0.015}"/>
-  </joint>
-  <joint name="rear_scanner_to_base_joint" type="fixed">
-    <parent link="base_link" />
-    <child link="rear_scanner_mount_link" />
-    <origin xyz="${-body_length/2 + 0.035} 0 ${body_height/2 - 0.015}" rpy="0 0 ${M_PI}"/>
-  </joint>
-  <joint name="pico_flexx_lense" type="fixed">
-    <parent link="pico_flexx_model_link" />
-    <child link="pico_flexx_optical_frame" />
-    <origin xyz="0.005 -0.009 0.002" rpy="${M_PI/2} 0 ${M_PI/2}"/>
   </joint>
   <link name="imu">

Commit message: fixed gazebo sim teleop

File: ceres_description/urdf/ceres.urdf.xacro (robot description, xacro)
@@ -23,10 +23,11 @@
   <xacro:property name="axis_left" value="${body_width/2 + wheel_body_offset}"/>
   <xacro:property name="axis_length" value="${body_width + 2 * wheel_body_offset}" />
-  <xacro:property name="turning_adaptation" value="0.95" />
+  <xacro:property name="turning_adaptation" value="0.2" />
+  <xacro:property name="torque" value="40.0" />
   <xacro:property name="bearing_width" value="0.05"/>
   <xacro:property name="bearing_height" value="0.09"/>
   <xacro:property name="bearing_thickness" value="0.01"/>
   <xacro:property name="body_mass" value="40.0"/>
-  <xacro:property name="wheel_mass" value="3.0"/>
+  <xacro:property name="wheel_mass" value="30.0"/>
   <xacro:property name="imu_width" value="0.036"/>
   <xacro:property name="imu_length" value="0.038"/>
@@ -235,6 +236,6 @@
       <wheel_separation>${axis_length}</wheel_separation>
       <wheel_diameter>${2*wheel_radius}</wheel_diameter>
-      <turning_adaptation>0.95</turning_adaptation>
-      <torque>4.0</torque>
+      <turning_adaptation>${turning_adaptation}</turning_adaptation>
+      <torque>${torque}</torque>
       <max_velocity>2</max_velocity>
       <updateRate>40.0</updateRate>
